File: hardware/cansult.kicad_pcb (KiCad board)
At the start: 4 copper layers, 44 x 34 mm, 69 parts, among them J1 X2016WV-06K-N0SN, J2 DEBUG, J3 Conn_01x02_Pin, J4 BT, Q1 2N7002, Q2 2N7002, U1 LM358, U2 MC74HC4060ADTR2G, U3 MCP2562-E-SN, U4 STM32F103T6U6A, U5 LD1117S33TR_SOT223, U6 LM78M05_TO252, Y1 4.9152 MHz, Y2 16MHz 9pF

Commit message: fix: use 12v fused; relink libs
Parts:
- TP1, TP2, TP3, TP4, TP5, TP6, TP7: footprint footprints:KEYSTONE_5015 -> local:KEYSTONE_5015
Connections:
- D2 pad 1: /power/+12 FUSED -> +12VF
- D3 pad 2: /power/+12 FUSED -> +12VF
- F1 pad 1: /power/+12 FUSED -> +12VF
- R5 pad 2: +12V -> +12VF
- R7 pad 2: +12V -> +12VF
Routing:
- net +12VF: track 0.00 -> 52.0 mm, vias 0 -> 3
- net +12V: track 37.5 -> 10.7 mm, vias 1 -> 0
- net /power/+12 FUSED: track 8.92 -> 0.00 mm
- net CNSLT_TX: track 19.3 -> 20.6 mm
- net GND: vias 116 -> 115

Commit message: prepare for production
Parts:
- C12, C7: footprint Capacitor_SMD:C_0805_2012Metric -> Capacitor_SMD:C_0603_1608Metric
- C3, C4: footprint Capacitor_SMD:C_0402_1005Metric -> Capacitor_SMD:C_0603_1608Metric
- F1: value 0805-FF PW 0A5 -> 0603 CP06V5TR50 500mA 50V; footprint Fuse:Fuse_0805_2012Metric -> Fuse:Fuse_0603_1608Metric
- moved Y1 0.61 mm to (168.8, 77.5)
- moved C3 0.30 mm to (172.5, 77.2)
- moved C4 0.30 mm to (172.5, 73.2)
Routing:
- net GND: track 80.7 -> 81.9 mm
- net OSC_IN: track 11.4 -> 12.3 mm
