File: hardware/cansult.kicad_pcb (KiCad board)
At the start: 4 copper layers, 44 x 34 mm, 69 parts, among them J1 X2016WV-06K-N0SN, J2 DEBUG, J3 Conn_01x02_Pin, J4 BT, Q1 2N7002, Q2 2N7002, U1 LM358, U2 MC74HC4060ADTR2G, U3 MCP2562-E-SN, U4 STM32F103T6U6A, U5 LD1117S33TR_SOT223, U6 LM78M05_TO252, Y1 4.9152 MHz, Y2 16MHz 9pF

Commit message: fix(uart): address UART drop root causes and add MCU temperature diag
Three firmware bugs uncovered during thermal investigation:

- ISR byte-stealing cascade: STM32F1 clears FE/NE/ORE only via SR+DR
  read; doing that in USART1_IRQHandler steals bytes from DMA and
  creates a self-sustaining framing error storm. Disable EIE after
  HAL_UART_Receive_DMA and poll error flags from cansult_tick() instead.
- ECU_INFO frame size was 24 (parser waited for a byte that never
  arrived); correct size is 23. Part-number offset adjusted to 18.
- WAITING_ECU_RESPONSE timeout fell back to STARTUP, re-running the
  full init handshake. Proceed to IDLE (streaming) instead.

Diagnostic infrastructure:

- Enable ADC1 on Temperature Sensor channel (ADC clock /6 = 12 MHz,
  239.5-cycle sample). readMcuTempC10() returns MCU die temp × 10.
- New 0x66B extended diag frame: FE/NE as full uint16, current MCU
  temp, and MCU temp captured at the moment of the first FE
  (read inline so the value isn't stale or BSS-zero).
- 0x665 bytes 1-3 now carry saturating per-second rates for ORE,
  FE+NE, and CAN failures (previous low-byte truncation silently
  lost data once counters grew to uint16). Byte 6 now carries
  reconnect_count, which is correctly counted on transitions into
  STARTUP (was incrementing every tick).

Python decoders updated for the new 0x665 semantics and 0x66B frame.

Thermal investigation conclusion: UART drops are caused by LDO/LMV358
heating (MCU die rises only ~1.6°C at failure onset, consistent with
the MCU being a proxy thermometer for the real hot components).
Cooling the board eliminates all UART errors (22 min clean across
two captures). Next step is hardware (switching regulator, heatsink,
or physical separation in next PCB revision).

Co-Authored-By: Claude Opus 4.6 (1M context) <noreply@anthropic.com>
Parts:
- U1: value LM358 -> LMV358
Changed lines of the file:
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@@
     (descr "SOIC, 8 Pin (JEDEC MS-012AA, https://www.analog.com/media/en/package-pcb-resources/package/pkg_pdf/soic_narrow-r/r_8.pdf), generated with kicad-footprint-generator ipc_gullwing_generator.py")
     (tags "SOIC SO")
-    (property "LCSC" "C7950")
+    (property "LCSC" "TBD_LMV358")
     (property "Sheetfile" "consult.kicad_sch")
     (property "Sheetname" "consult")
-    (property "ki_description" "Low-Power, Dual Operational Amplifiers, DIP-8/SOIC-8/TO-99-8")
+    (property "ki_description" "Rail-to-Rail Output Dual Operational Amplifier, 2.7V-5.5V, SOIC-8")
     (property "ki_keywords" "dual opamp")
     (attr smd)
@@
         (effects (font (size 1 1) (thickness 0.15)))
     )
-    (fp_text value "LM358" (at 0 3.4) (layer "F.Fab")
+    (fp_text value "LMV358" (at 0 3.4) (layer "F.Fab")
         (effects (font (size 1 1) (thickness 0.15)))
     )
