File: hardware/cansult.kicad_sch (KiCad schematic)
At the start: 2 parts

Commit message: prepare for production
Parts:
- H1, H2: LCSC (none) -> NA; now left out of the parts list
Changed lines of the file:
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@@
   (paper "A4")
   (symbol (lib_id "Mechanical:MountingHole") (at 27.94 100.33 0) (unit 1)
-    (in_bom yes) (on_board yes) (dnp no) (fields_autoplaced)
+    (in_bom no) (on_board yes) (dnp no) (fields_autoplaced)
     (property "Reference" "H2" (at 30.48 99.695 0)
       (effects (font (size 1.27 1.27)) (justify left))
@@
       (effects (font (size 1.27 1.27)) hide)
     )
+    (property "LCSC" "NA" (at 27.94 100.33 0)
+      (effects (font (size 1.27 1.27)) hide)
+    )
     (instances
       (project "cansult"
@@
   )
   (symbol (lib_id "Mechanical:MountingHole") (at 27.94 91.44 0) (unit 1)
-    (in_bom yes) (on_board yes) (dnp no) (fields_autoplaced)
+    (in_bom no) (on_board yes) (dnp no) (fields_autoplaced)
     (property "Reference" "H1" (at 30.48 90.805 0)
       (effects (font (size 1.27 1.27)) (justify left))
@@
       (effects (font (size 1.27 1.27)) hide)
     )
+    (property "LCSC" "NA" (at 27.94 91.44 0)
+      (effects (font (size 1.27 1.27)) hide)
+    )
