File: hardware/consult.kicad_sch (KiCad schematic)
At the start: 29 parts

Commit message: fix(uart): address UART drop root causes and add MCU temperature diag
Three firmware bugs uncovered during thermal investigation:

- ISR byte-stealing cascade: STM32F1 clears FE/NE/ORE only via SR+DR
  read; doing that in USART1_IRQHandler steals bytes from DMA and
  creates a self-sustaining framing error storm. Disable EIE after
  HAL_UART_Receive_DMA and poll error flags from cansult_tick() instead.
- ECU_INFO frame size was 24 (parser waited for a byte that never
  arrived); correct size is 23. Part-number offset adjusted to 18.
- WAITING_ECU_RESPONSE timeout fell back to STARTUP, re-running the
  full init handshake. Proceed to IDLE (streaming) instead.

Diagnostic infrastructure:

- Enable ADC1 on Temperature Sensor channel (ADC clock /6 = 12 MHz,
  239.5-cycle sample). readMcuTempC10() returns MCU die temp × 10.
- New 0x66B extended diag frame: FE/NE as full uint16, current MCU
  temp, and MCU temp captured at the moment of the first FE
  (read inline so the value isn't stale or BSS-zero).
- 0x665 bytes 1-3 now carry saturating per-second rates for ORE,
  FE+NE, and CAN failures (previous low-byte truncation silently
  lost data once counters grew to uint16). Byte 6 now carries
  reconnect_count, which is correctly counted on transitions into
  STARTUP (was incrementing every tick).

Python decoders updated for the new 0x665 semantics and 0x66B frame.

Thermal investigation conclusion: UART drops are caused by LDO/LMV358
heating (MCU die rises only ~1.6°C at failure onset, consistent with
the MCU being a proxy thermometer for the real hot components).
Cooling the board eliminates all UART errors (22 min clean across
two captures). Next step is hardware (switching regulator, heatsink,
or physical separation in next PCB revision).

Co-Authored-By: Claude Opus 4.6 (1M context) <noreply@anthropic.com>
Parts:
- U? (x3): value LM358 -> LMV358; symbol Amplifier_Operational:LM358 -> Amplifier_Operational:LMV358; LCSC C7950 -> TBD_LMV358
Changed lines of the file:
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@@
     )
   )
-  (symbol (lib_id "Amplifier_Operational:LM358") (at 62.23 36.83 0) (unit 2)
+  (symbol (lib_id "Amplifier_Operational:LMV358") (at 62.23 36.83 0) (unit 2)
     (in_bom yes) (on_board yes) (dnp no) (fields_autoplaced)
     (property "Reference" "U?" (at 62.23 27.94 0)
       (effects (font (size 1.27 1.27)))
     )
-    (property "Value" "LM358" (at 62.23 30.48 0)
+    (property "Value" "LMV358" (at 62.23 30.48 0)
       (effects (font (size 1.27 1.27)))
     )
@@
       (effects (font (size 1.27 1.27)) hide)
     )
-    (property "Datasheet" "http://www.ti.com/lit/ds/symlink/lm2904-n.pdf" (at 62.23 36.83 0)
-      (effects (font (size 1.27 1.27)) hide)
-    )
-    (property "LCSC" "C7950" (at 62.23 36.83 0)
+    (property "Datasheet" "https://www.ti.com/lit/ds/symlink/lmv358.pdf" (at 62.23 36.83 0)
+      (effects (font (size 1.27 1.27)) hide)
+    )
+    (property "LCSC" "TBD_LMV358" (at 62.23 36.83 0)
       (effects (font (size 1.27 1.27)) hide)
     )
@@
     )
   )
-  (symbol (lib_id "Amplifier_Operational:LM358") (at 62.23 55.88 0) (unit 1)
+  (symbol (lib_id "Amplifier_Operational:LMV358") (at 62.23 55.88 0) (unit 1)
     (in_bom yes) (on_board yes) (dnp no) (fields_autoplaced)
     (property "Reference" "U?" (at 62.23 46.99 0)
       (effects (font (size 1.27 1.27)))
     )
-    (property "Value" "LM358" (at 62.23 49.53 0)
+    (property "Value" "LMV358" (at 62.23 49.53 0)
       (effects (font (size 1.27 1.27)))
     )
@@
       (effects (font (size 1.27 1.27)) hide)
     )
-    (property "Datasheet" "http://www.ti.com/lit/ds/symlink/lm2904-n.pdf" (at 62.23 55.88 0)
-      (effects (font (size 1.27 1.27)) hide)
-    )
-    (property "LCSC" "C7950" (at 62.23 55.88 0)
+    (property "Datasheet" "https://www.ti.com/lit/ds/symlink/lmv358.pdf" (at 62.23 55.88 0)
+      (effects (font (size 1.27 1.27)) hide)
+    )
+    (property "LCSC" "TBD_LMV358" (at 62.23 55.88 0)
       (effects (font (size 1.27 1.27)) hide)
     )
@@
     )
   )
-  (symbol (lib_id "Amplifier_Operational:LM358") (at 102.87 50.8 0) (unit 3)
+  (symbol (lib_id "Amplifier_Operational:LMV358") (at 102.87 50.8 0) (unit 3)
     (in_bom yes) (on_board yes) (dnp no) (fields_autoplaced)
     (property "Reference" "U?" (at 101.6 50.165 0)
       (effects (font (size 1.27 1.27)) (justify left))
     )
-    (property "Value" "LM358" (at 101.6 52.705 0)
+    (property "Value" "LMV358" (at 101.6 52.705 0)
       (effects (font (size 1.27 1.27)) (justify left))
     )
@@
       (effects (font (size 1.27 1.27)) hide)
     )
-    (property "Datasheet" "http://www.ti.com/lit/ds/symlink/lm2904-n.pdf" (at 102.87 50.8 0)
-      (effects (font (size 1.27 1.27)) hide)
-    )
-    (property "LCSC" "C7950" (at 102.87 50.8 0)
-      (effects (font (size 1.27 1.27)) hide)
-    )
+    (property "Datasheet" "https://www.ti.com/lit/ds/symlink/lmv358.pdf" (at 102.87 50.8 0)
+      (effects (font (size 1.27 1.27)) hide)
+    )
+    (property "LCSC" "TBD_LMV358" (at 102.87 50.8 0)
+      (effects (font (size 1.27 1.27)) hide)
+    )
