File: hardware/power.kicad_sch (KiCad schematic)
At the start: 13 parts, among them U5 LD1117S33TR_SOT223, U6 LM78M05_TO252

Commit message: fix: use 12v fused; relink libs
Connections:
- net +12 FUSED renamed +12VF
Changed lines of the file:
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@@
+    (stroke (width 0) (type default))
+  )
+  (wire (pts (xy 64.77 43.18) (xy 64.77 45.72))
     (stroke (width 0) (type default))
   )
@@
     (effects (font (size 1.27 1.27)) (justify left bottom))
   )
-  (label "+12 FUSED" (at 66.04 45.72 0) (fields_autoplaced)
-    (effects (font (size 1.27 1.27)) (justify left bottom))
-  )
   (label "+12 VIN" (at 121.92 45.72 0) (fields_autoplaced)
     (effects (font (size 1.27 1.27)) (justify left bottom))
@@
     )
   )
+  (global_label "+12VF" (shape input) (at 64.77 43.18 90) (fields_autoplaced)
+    (effects (font (size 1.27 1.27)) (justify left))
+    (property "Intersheetrefs" "${INTERSHEET_REFS}" (at 64.77 34.0262 90)
+      (effects (font (size 1.27 1.27)) (justify left) hide)
+    )
+  )

Commit message: prepare for production
Parts:
- C20, C23, C24, C27: LCSC (none) -> C15849
- C21, C25, C26, C28: LCSC (none) -> C14663
- D2: LCSC (none) -> C133688
- D3: LCSC (none) -> C68337
- F1: value 0805-FF PW 0A5 -> 0603 CP06V5TR50 500mA 50V; footprint Fuse:Fuse_0805_2012Metric -> Fuse:Fuse_0603_1608Metric; LCSC C2977524 -> C163136
- U5: LCSC (none) -> C86781
Changed lines of the file:
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@@
     (stroke (width 0) (type default))
   )
-  (polyline (pts (xy 24.13 96.52) (xy 24.13 30.48))
+  (polyline (pts (xy 24.13 96.52) (xy 24.13 24.13))
     (stroke (width 0) (type default))
   )
@@
     (stroke (width 0) (type default))
   )
-  (polyline (pts (xy 193.04 30.48) (xy 193.04 96.52))
+  (polyline (pts (xy 193.04 24.13) (xy 193.04 96.52))
     (stroke (width 0) (type default))
   )
@@
     (stroke (width 0) (type default))
   )
-  (wire (pts (xy 64.77 43.18) (xy 64.77 45.72))
+  (wire (pts (xy 64.77 38.1) (xy 64.77 45.72))
     (stroke (width 0) (type default))
   )
@@
     (stroke (width 0) (type default))
   )
-  (polyline (pts (xy 24.13 30.48) (xy 193.04 30.48))
+  (polyline (pts (xy 24.13 24.13) (xy 193.04 24.13))
     (stroke (width 0) (type default))
   )
@@
     (effects (font (size 1.27 1.27)) (justify left bottom))
   )
-  (text "VIN to 5V" (at 38.1 29.21 0)
+  (text "VIN to 5V" (at 27.94 22.86 0)
     (effects (font (size 1.27 1.27)) (justify left bottom))
   )
@@
     )
   )
-  (global_label "+12VF" (shape input) (at 64.77 43.18 90) (fields_autoplaced)
+  (global_label "+12VF" (shape input) (at 64.77 38.1 90) (fields_autoplaced)
     (effects (font (size 1.27 1.27)) (justify left))
-    (property "Intersheetrefs" "${INTERSHEET_REFS}" (at 64.77 34.0262 90)
+    (property "Intersheetrefs" "${INTERSHEET_REFS}" (at 64.77 28.9462 90)
       (effects (font (size 1.27 1.27)) (justify left) hide)
     )
@@
       (effects (font (size 1.27 1.27)) hide)
     )
+    (property "LCSC" "C14663" (at 129.54 64.77 0)
+      (effects (font (size 1.27 1.27)) hide)
+    )
     (pin "1")
     (pin "2")
@@
   (symbol (lib_id "Device:Fuse") (at 54.61 45.72 270) (unit 1)
     (in_bom yes) (on_board yes) (dnp no)
-    (property "Reference" "F1" (at 54.61 40.7162 90)
-      (effects (font (size 1.27 1.27)))
-    )
-    (property "Value" "0805-FF PW 0A5" (at 54.61 43.0276 90)
-      (effects (font (size 1.27 1.27)))
-    )
-    (property "Footprint" "Fuse:Fuse_0805_2012Metric" (at 54.61 43.942 90)
+    (property "Reference" "F1" (at 54.61 48.26 90)
+      (effects (font (size 1.27 1.27)))
+    )
+    (property "Value" "0603 CP06V5TR50 500mA 50V" (at 48.26 41.91 90)
+      (effects (font (size 1.27 1.27)))
+    )
+    (property "Footprint" "Fuse:Fuse_0603_1608Metric" (at 54.61 43.942 90)
       (effects (font (size 1.27 1.27)) hide)
     )
@@
       (effects (font (size 1.27 1.27)) hide)
     )
-    (property "LCSC" "C2977524" (at 54.61 45.72 90)
+    (property "LCSC" "C163136" (at 54.61 45.72 90)
       (effects (font (size 1.27 1.27)) hide)
     )
@@
       (effects (font (size 1.27 1.27)) hide)
     )
+    (property "LCSC" "C15849" (at 63.5 125.73 0)
+      (effects (font (size 1.27 1.27)) hide)
+    )
     (pin "1")
     (pin "2")
@@
       (effects (font (size 1.27 1.27)) hide)
     )
+    (property "LCSC" "C14663" (at 139.7 125.73 0)
+      (effects (font (size 1.27 1.27)) hide)
+    )
     (pin "1")
     (pin "2")
@@
       (effects (font (size 1.27 1.27)) hide)
     )
+    (property "LCSC" "C86781" (at 101.6 118.11 0)
+      (effects (font (size 1.27 1.27)) hide)
+    )
     (pin "1")
     (pin "2")
@@
       (effects (font (size 1.27 1.27)) hide)
     )
+    (property "LCSC" "C15849" (at 157.48 64.77 0)
+      (effects (font (size 1.27 1.27)) hide)
+    )
     (pin "1")
     (pin "2")
@@
       (effects (font (size 1.27 1.27)) hide)
     )
+    (property "LCSC" "C68337" (at 90.17 45.72 0)
+      (effects (font (size 1.27 1.27)) hide)
+    )
     (pin "1")
     (pin "2")
@@
     )
     (property "Datasheet" "~" (at 115.57 64.77 0)
+      (effects (font (size 1.27 1.27)) hide)
+    )
+    (property "LCSC" "C15849" (at 115.57 64.77 0)
       (effects (font (size 1.27 1.27)) hide)
     )
@@
       (effects (font (size 1.27 1.27)) hide)
     )
+    (property "LCSC" "C133688" (at 64.77 64.77 0)
+      (effects (font (size 1.27 1.27)) hide)
+    )
     (pin "1")
     (pin "2")
@@
       (effects (font (size 1.27 1.27)) hide)
     )
+    (property "LCSC" "C14663" (at 83.82 125.73 0)
+      (effects (font (size 1.27 1.27)) hide)
+    )
     (pin "1")
     (pin "2")
@@
       (effects (font (size 1.27 1.27)) hide)
     )
+    (property "LCSC" "C14663" (at 171.45 64.77 0)
+      (effects (font (size 1.27 1.27)) hide)
+    )
     (pin "1")
     (pin "2")
@@
       (effects (font (size 1.27 1.27)) hide)
     )
+    (property "LCSC" "C15849" (at 119.38 125.73 0)
+      (effects (font (size 1.27 1.27)) hide)
+    )
